Commit message: Added gen3 simulation functionality
need to figure out how to isolate jaco2 vs gen2 in ada_description
need to correct angle for fork plus camera mount

File: ada_description/urdf/ada.xacro (robot description, xacro)
@@ -18,5 +18,6 @@
   <xacro:include filename="$(find ada_description)/urdf/forque/forque.xacro"/>
   <xacro:include filename="$(find ada_description)/urdf/camera/camera.xacro"/>
-  <xacro:include filename="$(find ada_description)/urdf/j2n6s200.xacro"/>
+  <!--xacro:include filename="$(find ada_description)/urdf/j2n6s200.xacro"/ gurnoork comment -->
+  <xacro:include filename="$(find kortex_description)/robots/kortex_robot.xacro"/>
   <xacro:arg
     name="use_forque"
@@ -53,7 +54,40 @@
     value="root_tilt"
   />
-  <xacro:j2n6s200 base_parent="${robot_root}"/>
+  <!--xacro:j2n6s200 base_parent="${robot_root}"/-->
+  <xacro:load_robot
+    parent="${robot_root}"
+    arm="gen3"
+    dof="7"
+    prefix="ada_"
+    gripper=""
+    gripper_joint_name="finger_joint"
+    gripper_max_velocity="100.0"
+    gripper_max_force="100.0"
+    vision="true"
+    robot_ip="192.168.11.11"
+    username="admin"
+    password="admin"
+    port="10000"
+    port_realtime="10001"
+    session_inactivity_timeout_ms="60000"
+    connection_inactivity_timeout_ms="2000"
+    use_internal_bus_gripper_comm="false"
+    use_fake_hardware="true"
+    fake_sensor_commands="false"
+    sim_gazebo="false"
+    sim_ignition="false"
+    sim_isaac="false"
+    use_external_cable="false"
+    initial_positions="${xacro.load_yaml('$(find kortex_description)/config/initial_positions.yaml')}"
+    moveit_active="true">
+    <origin xyz="0 0 0" rpy="0 0 0"/>
+  </xacro:load_robot>
+  <!--xacro:camera_assembly
+    base_parent="j2n6s200_link_6"
+    base_xyz="0.0165 0 0.0011"
+    base_rpy="${3*J_PI/2} 0 ${3*J_PI/2}"
+  / gurnoork comment -->
   <xacro:camera_assembly
-    base_parent="j2n6s200_link_6"
+    base_parent="ada_end_effector_link"
     base_xyz="0.0165 0 0.0011"
     base_rpy="${3*J_PI/2} 0 ${3*J_PI/2}"
@@ -96,5 +130,5 @@
     />
   </xacro:forque_assembly_link>
-  <xacro:forque_assembly_joint
+  <!--xacro:forque_assembly_joint
     joint_name="FTArmMount_to_arm"
     parent="j2n6s200_link_6"
@@ -102,6 +136,28 @@
     joint_origin_xyz="0.0065 -0.011 -0.0075"
     joint_origin_rpy="${J_PI/2} 0 ${J_PI/2}"
+  /-->
+  <xacro:forque_assembly_joint
+    joint_name="FTArmMount_to_arm"
+    parent="ada_end_effector_link"
+    child="FTArmMount"
+    joint_origin_xyz="0.0065 -0.011 -0.0075"
+    joint_origin_rpy="${3*J_PI/2} 0 ${J_PI/2}"
   />
   <xacro:if value="$(arg use_forque)">
+    <xacro:forque_assembly base_parent="FTArmMount"/>
+    <link name="FTSensor"/>
+    <joint
+      name="EE_to_FTSensor"
+      type="fixed"
+    >
+      <child link="FTSensor"/>
+      <parent link="ada_end_effector_link"/> <!-- gurnoork might have to be actual endeffector? or FTArmMount -->
+      <origin
+        rpy="0 0 0"
+        xyz="0.0 0.0 0.092"
+      />
+    </joint>
+  </xacro:if>
+  <!--xacro:if value="$(arg use_forque)">
     <xacro:forque_assembly base_parent="FTArmMount"/>
     <link name="FTSensor"/>
@@ -117,4 +173,4 @@
       />
     </joint>
-  </xacro:if>
+  </xacro:if-->
 </robot>

File: ada_description/urdf/ada_gen2.xacro (robot description, xacro)
@@ -18,6 +18,5 @@
   <xacro:include filename="$(find ada_description)/urdf/forque/forque.xacro"/>
   <xacro:include filename="$(find ada_description)/urdf/camera/camera.xacro"/>
-  <!--xacro:include filename="$(find ada_description)/urdf/j2n6s200.xacro"/ gurnoork comment -->
-  <xacro:include filename="$(find kortex_description)/robots/kortex_robot.xacro"/>
+  <xacro:include filename="$(find ada_description)/urdf/j2n6s200.xacro"/>
   <xacro:arg
     name="use_forque"
@@ -54,40 +53,7 @@
     value="root_tilt"
   />
-  <!--xacro:j2n6s200 base_parent="${robot_root}"/-->
-  <xacro:load_robot
-    parent="${robot_root}"
-    arm="gen3"
-    dof="7"
-    prefix="ada_"
-    gripper=""
-    gripper_joint_name="finger_joint"
-    gripper_max_velocity="100.0"
-    gripper_max_force="100.0"
-    vision="true"
-    robot_ip="192.168.11.11"
-    username="admin"
-    password="admin"
-    port="10000"
-    port_realtime="10001"
-    session_inactivity_timeout_ms="60000"
-    connection_inactivity_timeout_ms="2000"
-    use_internal_bus_gripper_comm="false"
-    use_fake_hardware="true"
-    fake_sensor_commands="false"
-    sim_gazebo="false"
-    sim_ignition="false"
-    sim_isaac="false"
-    use_external_cable="false"
-    initial_positions="${xacro.load_yaml('$(find kortex_description)/config/initial_positions.yaml')}"
-    moveit_active="true">
-    <origin xyz="0 0 0" rpy="0 0 0"/>
-  </xacro:load_robot>
-  <!--xacro:camera_assembly
+  <xacro:j2n6s200 base_parent="${robot_root}"/>
+  <xacro:camera_assembly
     base_parent="j2n6s200_link_6"
-    base_xyz="0.0165 0 0.0011"
-    base_rpy="${3*J_PI/2} 0 ${3*J_PI/2}"
-  / gurnoork comment -->
-  <xacro:camera_assembly
-    base_parent="ada_end_effector_link"
     base_xyz="0.0165 0 0.0011"
     base_rpy="${3*J_PI/2} 0 ${3*J_PI/2}"
@@ -130,5 +96,5 @@
     />
   </xacro:forque_assembly_link>
-  <!--xacro:forque_assembly_joint
+  <xacro:forque_assembly_joint
     joint_name="FTArmMount_to_arm"
     parent="j2n6s200_link_6"
@@ -136,28 +102,6 @@
     joint_origin_xyz="0.0065 -0.011 -0.0075"
     joint_origin_rpy="${J_PI/2} 0 ${J_PI/2}"
-  /-->
-  <xacro:forque_assembly_joint
-    joint_name="FTArmMount_to_arm"
-    parent="ada_end_effector_link"
-    child="FTArmMount"
-    joint_origin_xyz="0.0065 -0.011 -0.0075"
-    joint_origin_rpy="${3*J_PI/2} 0 ${J_PI/2}"
   />
   <xacro:if value="$(arg use_forque)">
-    <xacro:forque_assembly base_parent="FTArmMount"/>
-    <link name="FTSensor"/>
-    <joint
-      name="EE_to_FTSensor"
-      type="fixed"
-    >
-      <child link="FTSensor"/>
-      <parent link="ada_end_effector_link"/> <!-- gurnoork might have to be actual endeffector? or FTArmMount -->
-      <origin
-        rpy="0 0 0"
-        xyz="0.0 0.0 0.092"
-      />
-    </joint>
-  </xacro:if>
-  <!--xacro:if value="$(arg use_forque)">
     <xacro:forque_assembly base_parent="FTArmMount"/>
     <link name="FTSensor"/>
@@ -173,4 +117,4 @@
       />
     </joint>
-  </xacro:if-->
+  </xacro:if>
 </robot>

File: ada_moveit_kortex/config/ada.kortex.urdf.xacro (robot description, xacro)
@@ -13,5 +13,5 @@
   />
   <!-- Import ada urdf file -->
-  <xacro:include filename="$(find ada_description)/urdf/ada_kortex.xacro"/>
+  <xacro:include filename="$(find ada_description)/urdf/ada.xacro"/>
   <!-- Import control_xacro -->
   <xacro:include filename="ada.ros2_control.xacro"/>
