Commit message: Testing camera calibration for gen3

File: ada_description/urdf/ada.gen3.xacro (robot description, xacro)
@@ -64,5 +64,5 @@
     gripper_max_force="100.0"
     vision="true"
-    robot_ip="192.168.11.11"
+    robot_ip="192.168.1.10"
     username="admin"
     password="admin"
@@ -72,5 +72,5 @@
     connection_inactivity_timeout_ms="2000"
     use_internal_bus_gripper_comm="false"
-    use_fake_hardware="true"
+    use_fake_hardware="false"
     fake_sensor_commands="false"
     sim_gazebo="false"

File: ada_description/urdf/ada.xacro (robot description, xacro)
@@ -22,4 +22,8 @@
     name="use_forque"
     default="true"
+  />
+  <xacro:arg
+    name="use_fake_hardware"
+    default="false"
   />
   <link name="root"/>
@@ -64,5 +68,5 @@
     gripper_max_force="100.0"
     vision="true"
-    robot_ip="192.168.11.11"
+    robot_ip="192.168.1.10"
     username="admin"
     password="admin"
@@ -72,5 +76,5 @@
     connection_inactivity_timeout_ms="2000"
     use_internal_bus_gripper_comm="false"
-    use_fake_hardware="true"
+    use_fake_hardware="$(arg use_fake_hardware)"
     fake_sensor_commands="false"
     sim_gazebo="false"
@@ -80,5 +84,5 @@
     initial_positions="${xacro.load_yaml('$(find kortex_description)/config/initial_positions.yaml')}"
     moveit_active="true">
-    <origin xyz="0 0 0" rpy="0 0 0"/>
+    <origin xyz="0 -0.20 0.13" rpy="0 0 0"/>
   </xacro:load_robot>
   <!--xacro:camera_assembly

File: ada_description/urdf/ada_expanded.urdf (robot description, URDF)
Before this commit: robot ada, 35 links, 34 joints
Joints:
- joint ada_base_joint: origin xyz=0 0 0 rpy=0 0 0 -> xyz=0 -0.20 0.13 rpy=0 0 0

File: ada_moveit/config/ada.ros2_control.xacro (robot description, xacro)
@@ -3,5 +3,5 @@
   <xacro:macro
     name="ada_ros2_control"
-    params="name initial_positions_file sim"
+    params="name initial_positions_file sim robot_ip"
   >
     <xacro:property
@@ -30,4 +30,5 @@
         <xacro:if value="${sim == 'real'}">
           <plugin>ada_hardware/Gen3</plugin>
+          <param name="robot_ip">${robot_ip}</param>
         </xacro:if>
       </hardware>

File: ada_moveit/config/ada.urdf.xacro (robot description, xacro)
@@ -12,18 +12,27 @@
     default="real"
   />
+  <xacro:arg
+    name="robot_ip"
+    default="192.168.1.10"
+  />
+  <xacro:arg
+    name="use_fake_hardware"
+    default="${'$(arg sim)' != 'real'}"
+  />
   <!-- Import ada urdf file -->
   <xacro:include filename="$(find ada_description)/urdf/ada.xacro"/>
   <!-- Import control_xacro -->
   <xacro:include filename="ada.ros2_control.xacro"/>
-  <!-- Only add the ADAHardware ros2_control for real hardware.
-       For mock/mock_kortex, the Kortex hardware interface (ada_KortexMultiInterfaceHardware)
-       from ada_description already provides fake hardware support.
+  <!-- Only add the ADAHardware ros2_control for simulation modes.
+       For real hardware (sim='real'), KortexMultiInterfaceHardware from ada_description
+       handles the robot when use_fake_hardware=false.
        Adding both causes duplicate interface registration. -->
-  <xacro:if value="${'$(arg sim)' == 'real'}">
+  <xacro:unless value="${'$(arg sim)' == 'real'}">
     <xacro:ada_ros2_control
       name="ADAHardware"
       initial_positions_file="$(arg initial_positions_file)"
       sim="$(arg sim)"
+      robot_ip="$(arg robot_ip)"
     />
-  </xacro:if>
+  </xacro:unless>
 </robot>

File: kortex_description/robots/gen3.xacro (robot description, xacro)
@@ -5,5 +5,5 @@
     <xacro:arg name="dof" default="" />
     <xacro:arg name="vision" default="false" />
-    <xacro:arg name="robot_ip" default="192.168.11.11" />
+    <xacro:arg name="robot_ip" default="192.168.1.10" />
     <xacro:arg name="username" default="admin" />
     <xacro:arg name="password" default="admin" />

File: kortex_description/robots/kinova.urdf.xacro (robot description, xacro)
@@ -8,5 +8,5 @@
   <xacro:arg name="dof" default="7" />
   <xacro:arg name="vision" default="false" />
-  <xacro:arg name="robot_ip" default="192.168.11.11" />
+  <xacro:arg name="robot_ip" default="192.168.1.10" />
   <xacro:arg name="username" default="admin" />
   <xacro:arg name="password" default="admin" />
