Commit message: Cleaning up Gen3 Integration

File: ada_moveit/config/ada.ros2_control.xacro (robot description, xacro)
@@ -20,17 +20,17 @@
         </xacro:if>
         <xacro:if value="${sim == 'isaac'}">
-          <plugin>ada_hardware/JacoIsaac</plugin>
+          <plugin>ada_hardware/Gen3Isaac</plugin>
           <param name="namespace">/simulation</param>
         </xacro:if>
         <xacro:if value="${sim == 'real'}">
-          <plugin>ada_hardware/Jaco2</plugin>
+          <plugin>ada_hardware/Gen3</plugin>
         </xacro:if>
       </hardware>
-      <joint name="j2n6s200_joint_1">
+      <joint name="ada_joint_1">
         <command_interface name="position"/>
         <command_interface name="velocity"/>
         <command_interface name="effort"/>
         <state_interface name="position">
-          <param name="initial_value">${initial_positions['j2n6s200_joint_1']}</param>
+          <param name="initial_value">${initial_positions['joint_1']}</param>
         </state_interface>
         <state_interface name="velocity">
@@ -41,10 +41,10 @@
         </state_interface>
       </joint>
-      <joint name="j2n6s200_joint_2">
+      <joint name="ada_joint_2">
         <command_interface name="position"/>
         <command_interface name="velocity"/>
         <command_interface name="effort"/>
         <state_interface name="position">
-          <param name="initial_value">${initial_positions['j2n6s200_joint_2']}</param>
+          <param name="initial_value">${initial_positions['joint_2']}</param>
         </state_interface>
         <state_interface name="velocity">
@@ -55,10 +55,10 @@
         </state_interface>
       </joint>
-      <joint name="j2n6s200_joint_3">
+      <joint name="ada_joint_3">
         <command_interface name="position"/>
         <command_interface name="velocity"/>
         <command_interface name="effort"/>
         <state_interface name="position">
-          <param name="initial_value">${initial_positions['j2n6s200_joint_3']}</param>
+          <param name="initial_value">${initial_positions['joint_3']}</param>
         </state_interface>
         <state_interface name="velocity">
@@ -69,10 +69,10 @@
         </state_interface>
       </joint>
-      <joint name="j2n6s200_joint_4">
+      <joint name="ada_joint_4">
         <command_interface name="position"/>
         <command_interface name="velocity"/>
         <command_interface name="effort"/>
         <state_interface name="position">
-          <param name="initial_value">${initial_positions['j2n6s200_joint_4']}</param>
+          <param name="initial_value">${initial_positions['joint_4']}</param>
         </state_interface>
         <state_interface name="velocity">
@@ -83,10 +83,10 @@
         </state_interface>
       </joint>
-      <joint name="j2n6s200_joint_5">
+      <joint name="ada_joint_5">
         <command_interface name="position"/>
         <command_interface name="velocity"/>
         <command_interface name="effort"/>
         <state_interface name="position">
-          <param name="initial_value">${initial_positions['j2n6s200_joint_5']}</param>
+          <param name="initial_value">${initial_positions['joint_5']}</param>
         </state_interface>
         <state_interface name="velocity">
@@ -97,10 +97,10 @@
         </state_interface>
       </joint>
-      <joint name="j2n6s200_joint_6">
+      <joint name="ada_joint_6">
         <command_interface name="position"/>
         <command_interface name="velocity"/>
         <command_interface name="effort"/>
         <state_interface name="position">
-          <param name="initial_value">${initial_positions['j2n6s200_joint_6']}</param>
+          <param name="initial_value">${initial_positions['joint_6']}</param>
         </state_interface>
         <state_interface name="velocity">
@@ -111,24 +111,10 @@
         </state_interface>
       </joint>
-      <joint name="j2n6s200_joint_finger_1">
+      <joint name="ada_joint_7">
         <command_interface name="position"/>
         <command_interface name="velocity"/>
         <command_interface name="effort"/>
         <state_interface name="position">
-          <param name="initial_value">${initial_positions['j2n6s200_joint_finger_1']}</param>
-        </state_interface>
-        <state_interface name="velocity">
-          <param name="initial_value">0.0</param>
-        </state_interface>
-        <state_interface name="effort">
-          <param name="initial_value">0.0</param>
-        </state_interface>
-      </joint>
-      <joint name="j2n6s200_joint_finger_2">
-        <command_interface name="position"/>
-        <command_interface name="velocity"/>
-        <command_interface name="effort"/>
-        <state_interface name="position">
-          <param name="initial_value">${initial_positions['j2n6s200_joint_finger_2']}</param>
+          <param name="initial_value">${initial_positions['joint_7']}</param>
         </state_interface>
         <state_interface name="velocity">
