Commit message: plugin changed to add Gen3 option,

File: ada_hardware/urdf/ada_hardware.ros2_control.xacro (robot description, xacro)
@@ -3,5 +3,5 @@
   <xacro:macro
     name="ada_hardware_interface"
-    params="name prefix:=j2n6s200 sim readonly:=false"
+    params="name prefix:=ada sim readonly:=false"
   >
     <ros2_control
@@ -20,4 +20,7 @@
         </xacro:if>
         <xacro:if value="${sim == 'none'}">
+          <plugin>ada_hardware/Gen3</plugin>
+        </xacro:if>
+        <xacro:if value="${sim == 'Jaco2'}">
           <plugin>ada_hardware/Jaco2</plugin>
         </xacro:if>
@@ -84,4 +87,14 @@
         <state_interface name="effort"/>
       </joint>
+      <joint name="${prefix}_joint_7">
+        <xacro:unless value="${readonly}">
+          <command_interface name="position"/>
+          <command_interface name="velocity"/>
+          <command_interface name="effort"/>
+        </xacro:unless>
+        <state_interface name="position"/>
+        <state_interface name="velocity"/>
+        <state_interface name="effort"/>
+      </joint>
       <!-- Finger DOFs -->
       <joint name="${prefix}_joint_finger_1">
